File: Hardware/main_pcb/schemat.kicad_pcb (KiCad board)
At the start: 4 copper layers, 139.7 x 41.3 mm, 74 parts, among them J1 Battery, J10 Conn_Moto1_B, J11 Conn_Encoder2, J12 Conn_Moto1_A, J13 Conn_Moto1_B, J2 Conn_01x04_Socket, J3 SENSOR_CONN, J4 FTSH-105-01-F-DV-P-TR, J6 Conn_Encoder1, J9 Conn_Moto1_A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

Commit message: Minor fixes in schematics, added gerbers and schematics pdfs
Connections:
- U2 pad 35: /schemat_1/ENCODER1_CH1 -> unconnected-(U2-PB14-Pad35)
- U2 pad 37: unconnected-(U2-PC6-Pad37) -> /schemat_1/ENCODER1_CH1
Routing:
- net /schemat_1/ENCODER1_CH1: track 33.5 -> 34.5 mm
Changed lines of the file:
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@@
 	(net 69 "unconnected-(S1-Pad4)")
 	(net 70 "unconnected-(S1-Pad1)")
-	(net 71 "unconnected-(U2-PC6-Pad37)")
+	(net 71 "unconnected-(U2-PB14-Pad35)")
 	(net 72 "unconnected-(U2-PA12-Pad45)")
 	(net 73 "unconnected-(U2-PC12-Pad53)")
@@
 	(net 81 "/schemat_1/ENCODER2_ZERO")
 	(net 82 "/schemat_1/ENCODER1_ZERO")
-	(net 83 "unconnected-(Y2-NC-Pad2)")
-	(net 84 "unconnected-(Y2-NC-Pad4)")
+	(net 83 "unconnected-(Y1-NC-Pad2)")
+	(net 84 "unconnected-(Y1-NC-Pad4)")
 	(footprint "Resistor_SMD:R_0603_1608Metric_Pad0.98x0.95mm_HandSolder"
 		(layer "F.Cu")
@@
 			(layers "F.Cu" "F.Paste" "F.Mask")
 			(roundrect_rratio 0.25)
-			(net 49 "/schemat_1/ENCODER1_CH1")
+			(net 71 "unconnected-(U2-PB14-Pad35)")
 			(pinfunction "PB14")
-			(pintype "bidirectional")
+			(pintype "bidirectional+no_connect")
 		)
 		(pad "36" smd roundrect
@@
 			(layers "F.Cu" "F.Paste" "F.Mask")
 			(roundrect_rratio 0.25)
-			(net 71 "unconnected-(U2-PC6-Pad37)")
+			(net 49 "/schemat_1/ENCODER1_CH1")
 			(pinfunction "PC6")
-			(pintype "bidirectional+no_connect")
+			(pintype "bidirectional")
 		)
 		(pad "38" smd roundrect
@@
 			(size 1.2 1.4)
 			(layers "F.Cu" "F.Paste" "F.Mask")
-			(net 83 "unconnected-(Y2-NC-Pad2)")
+			(net 83 "unconnected-(Y1-NC-Pad2)")
 			(pinfunction "NC")
 			(pintype "no_connect")
@@
 			(size 1.2 1.4)
 			(layers "F.Cu" "F.Paste" "F.Mask")
-			(net 84 "unconnected-(Y2-NC-Pad4)")
+			(net 84 "unconnected-(Y1-NC-Pad4)")
 			(pinfunction "NC")
 			(pintype "no_connect")
@@
 	)
 	(segment
+		(start 138.3 115.1)
+		(end 139.71802 115.1)
+		(width 0.2)
+		(layer "F.Cu")
+		(net 6)
+	)
+	(segment
 		(start 131.1 106)
 		(end 122.375 106)
@@
 	)
 	(segment
-		(start 139.42042 115.3976)
+		(start 139.71802 115.1)
 		(end 140.396179 114.421841)
 		(width 0.2)
@@
 	)
 	(segment
-		(start 137.2 115.3976)
-		(end 139.42042 115.3976)
+		(start 138.0548 114.8548)
+		(end 138.3 115.1)
+		(width 0.2)
+		(layer "F.Cu")
+		(net 6)
+	)
+	(segment
+		(start 136.9 114.8548)
+		(end 138.0548 114.8548)
 		(width 0.2)
 		(layer "F.Cu")
@@
 	)
 	(via
-		(at 137.2 115.3976)
+		(at 136.9 114.8548)
 		(size 0.5)
 		(drill 0.25)
@@
 	)
 	(segment
-		(start 132.6 111.8976)
-		(end 132.6 111.3)
+		(start 135.5572 114.8548)
+		(end 132.6 111.8976)
 		(width 0.2)
 		(layer "B.Cu")
@@
 	)
 	(segment
-		(start 137.2 115.3976)
-		(end 136.1 115.3976)
+		(start 132.6 111.8976)
+		(end 132.6 111.3)
 		(width 0.2)
 		(layer "B.Cu")
@@
 	)
 	(segment
-		(start 136.1 115.3976)
-		(end 132.6 111.8976)
+		(start 136.9 114.8548)
+		(end 135.5572 114.8548)
 		(width 0.2)
 		(layer "B.Cu")
@@
 	)
 	(segment
-		(start 132.6 112.3)
-		(end 116.6 112.3)
+		(start 116.6 112.3)
+		(end 132.6 112.3)
 		(width 0.3)
 		(layer "F.Cu")
@@
 	)
 	(segment
-		(start 135.1 114.8)
-		(end 132.6 112.3)
+		(start 135.802401 115.502401)
+		(end 140.022725 115.502401)
 		(width 0.3)
 		(layer "F.Cu")
@@
 	)
 	(segment
-		(start 139.310912 114.8)
-		(end 135.1 114.8)
+		(start 140.022725 115.502401)
+		(end 140.749732 114.775394)
 		(width 0.3)
 		(layer "F.Cu")
@@
 	)
 	(segment
-		(start 140.042625 114.068287)
-		(end 139.310912 114.8)
+		(start 132.6 112.3)
+		(end 135.802401 115.502401)
 		(width 0.3)
 		(layer "F.Cu")
