File: Hardware/main_pcb/schemat_1.kicad_sch (KiCad schematic)
At the start: 64 parts, among them J1 Battery, J10 Conn_Moto1_B, J11 Conn_Encoder2, J12 Conn_Moto1_A, J13 Conn_Moto1_B, J2 Conn_01x04_Socket, J3 SENSOR_CONN, J4 FTSH-105-01-F-DV-P-TR, J6 Conn_Encoder1, J9 Conn_Moto1_A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

Commit message: Minor fixes in schematics, added gerbers and schematics pdfs
Connections:
- net ENCODER1_CH1: now also U2.37 (PC6); no longer U2.35 (PB14)
- no-connect marks 13 -> 12
Changed lines of the file:
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@@
 	(generator "eeschema")
 	(generator_version "8.0")
-	(paper "User" 522.656 239.801)
+	(paper "User" 370.256 239.801)
 	(junction
 		(at 191.77 213.36)
@@
 	)
 	(no_connect
-		(at 135.89 173.99)
-	)
-	(no_connect
-		(at 74.93 146.05)
-	)
-	(no_connect
 		(at 59.69 55.88)
 	)
@@
 	)
 	(no_connect
+		(at 110.49 189.23)
+	)
+	(no_connect
 		(at 59.69 30.48)
 	)
@@
 	(wire
 		(pts
-			(xy 110.49 189.23) (xy 116.84 189.23)
-		)
-		(stroke
-			(width 0)
-			(type default)
-		)
-	)
-	(wire
-		(pts
 			(xy 252.73 190.5) (xy 256.54 190.5)
 		)
@@
 	(wire
 		(pts
+			(xy 68.58 146.05) (xy 74.93 146.05)
+		)
+		(stroke
+			(width 0)
+			(type default)
+		)
+	)
+	(wire
+		(pts
 			(xy 262.89 88.9) (xy 262.89 91.44)
 		)
@@
 		)
 	)
-	(text_box "POWER"
+	(text_box "POWER SUPPLY"
 		(exclude_from_sim no)
 		(at 13.97 15.24 0)
@@
 		)
 	)
+	(label "ENCODER1_CH1"
+		(at 68.58 146.05 180)
+		(fields_autoplaced yes)
+		(effects
+			(font
+				(size 1.27 1.27)
+			)
+			(justify right bottom)
+		)
+	)
 	(label "LED3"
 		(at 116.84 184.15 0)
@@
 		(fields_autoplaced yes)
 		(effects
-			(font
-				(size 1.27 1.27)
-			)
-			(justify left bottom)
-		)
-	)
-	(label "ENCODER1_CH1"
-		(at 116.84 189.23 0)
-		(fields_autoplaced yes)
-		(effects
